File: led_watch.sch (KiCad schematic (older format))
At the start: 87 parts, among them J1 Conn_01x02, J2 Conn_01x02, SW1 SW_Push, U1 ATMEGA328P-AU, U2 MCP7940N, Y1 16MHz, Y2 32.768kHz

Commit message: "holy s#@% it's friday" commit
Parts:
- J3: renamed from J?; footprint (none) -> Pin_Headers:Pin_Header_Straight_1x02_Pitch1.00mm
Changed lines of the file:
@@
 $EndComp
 $Comp
-L GND #PWR05
+L GND #PWR01
 U 1 1 5AC3486C
 P 1000 1550
-F 0 "#PWR05" H 1000 1300 50  0001 C CNN
+F 0 "#PWR01" H 1000 1300 50  0001 C CNN
 F 1 "GND" H 1000 1400 50  0000 C CNN
 F 2 "" H 1000 1550 50  0001 C CNN
@@
 $EndComp
 $Comp
-L GND #PWR06
+L GND #PWR02
 U 1 1 5AC358D6
 P 3300 1700
-F 0 "#PWR06" H 3300 1450 50  0001 C CNN
+F 0 "#PWR02" H 3300 1450 50  0001 C CNN
 F 1 "GND" H 3300 1550 50  0000 C CNN
 F 2 "" H 3300 1700 50  0001 C CNN
@@
 	9800 2950 6450 2950
 $Comp
-L Conn_01x02 J?
+L Conn_01x02 J3
 U 1 1 5AF6672A
 P 4800 5050
-F 0 "J?" H 4800 5150 50  0000 C CNN
+F 0 "J3" H 4800 5150 50  0000 C CNN
 F 1 "Conn_01x02" H 4800 4850 50  0000 C CNN
-F 2 "" H 4800 5050 50  0001 C CNN
+F 2 "Pin_Headers:Pin_Header_Straight_1x02_Pitch1.00mm" H 4800 5050 50  0001 C CNN
 F 3 "" H 4800 5050 50  0001 C CNN
 	1    4800 5050
